File: pcb/p2000t-video-to-vga-adapter.kicad_pcb (KiCad board)
At the start: 2 copper layers, 81.3 x 68.6 mm, 40 parts, among them J1 DIN-6, J2 P2000T RAW, J3 P2000T CLEANED, J4 VGA, J5 VGA, SW1 SW_Push, U1 74LVC1G14, U2 74LVC1G14, U3 74LVC1G14, U4 74LVC1G14

Commit message: Interim commit firmware
Parts:
- SW1: value SW_Push -> RESET
- moved H1 2.29 mm to (115.8, 52.1)
- moved H3 2.29 mm to (115.8, 113.0)
- moved J5 2.29 mm to (111.8, 75.9)
- moved R21 0.92 mm to (136.3, 68.6)
- moved R24 0.92 mm to (136.3, 66.0)
- moved R25 0.92 mm to (136.3, 61.0)
- moved R27 0.92 mm to (136.3, 58.4)
- moved R31 0.92 mm to (136.3, 81.3)
- moved R33 0.92 mm to (136.3, 78.7)
- moved R34 0.92 mm to (136.3, 99.1)
- moved R35 0.92 mm to (136.3, 73.7)
- moved R37 0.92 mm to (136.3, 96.5)
- moved R38 0.92 mm to (136.3, 71.1)
- moved R39 0.92 mm to (136.3, 94.0)
- moved R40 0.92 mm to (136.3, 91.4)
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Routing:
- net +3V3: track 36.5 -> 102.9 mm
- net GND: track 259.1 -> 276.1 mm, vias 2 -> 4
- net R: track 57.4 -> 63.3 mm
- net B: track 41.2 -> 45.2 mm
- net IN_BLUE: track 47.0 -> 43.3 mm
- net IN_RED: track 32.0 -> 28.8 mm
- net H: track 44.6 -> 47.7 mm
- net G: track 48.9 -> 51.4 mm
- net V: track 45.5 -> 48.0 mm
- net SYNC: track 25.4 -> 27.2 mm, vias 0 -> 1
- net ~{IN_RED}: track 33.5 -> 32.0 mm
- net VGA_VSYNC: track 5.80 -> 6.72 mm
- net VGA_R3: track 5.80 -> 6.72 mm
- net VGA_R2: track 6.60 -> 7.53 mm
- net VGA_R1: track 6.60 -> 7.53 mm
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Other:
- board size 81.3 x 68.6 mm -> 83.6 x 68.6 mm
- board text added: "Philips P2000T Video Adapter v1.0"
- board text added: "S"
- board text added: "https://github.com/ifilot/p2000t-video-to-vga-adapter"
- board text removed: "Philips P2000M Video Adapter v1.1"
- board text removed: "Raw P2000T video signal"
- board text removed: "https://github.com/ifilot/p2000m-video-to-vga-adapter"
