File: pcb/p2000t-video-to-vga-adapter.kicad_pcb (KiCad board)
At the start: 2 copper layers, 83.6 x 68.6 mm, 40 parts, among them J1 DIN-6, J2 P2000T RAW, J3 P2000T CLEANED, J4 VGA, J5 VGA, SW1 RESET, U1 74LVC1G14, U2 74LVC1G14, U3 74LVC1G14, U4 74LVC1G14

Commit message: Fixing LICENSE details, polishing README.md, updating version
Other:
- board text added: "Licensed under CERN-OHL-S v2 https://github.com/ifilot/p2000t-video-to-vga-adapter"
- board text removed: "https://github.com/ifilot/p2000t-video-to-vga-adapter"
Changed lines of the file:
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@@
 		(layer "Edge.Cuts")
 	)
-	(gr_text "https://github.com/ifilot/p2000t-video-to-vga-adapter"
+	(gr_text "Licensed under CERN-OHL-S v2\nhttps://github.com/ifilot/p2000t-video-to-vga-adapter"
 		(at 141.605 115.57 0)
 		(layer "F.SilkS")
