File: pcb/p2000t-video-to-vga-adapter.kicad_sch (KiCad schematic)
At the start: 40 parts, among them J1 DIN-6, J2 P2000T RAW, J3 P2000T CLEANED, J4 VGA, J5 VGA, SW1 SW_Push, U1 74LVC1G14, U2 74LVC1G14, U3 74LVC1G14, U4 74LVC1G14

Commit message: Interim commit firmware
Parts:
- SW1: value SW_Push -> RESET
Other:
- note added: "Pico 2 controller: GPIO16-19 capture conditioned RGBS. GPIO0-11 provide 4-bit-per-channel RGB VGA output, with GPIO12-13 generating VGA sync. RUN has a manual reset switch; unused control, ADC, and GPIO pins are left unconnected."
- note removed: "Pico 2 controller: GPIO16-18 capture conditioned RGBS. GPIO0-11 provide 4-bit-per-channel RGB VGA output, with GPIO12-13 generating VGA sync. RUN has a manual reset switch; unused control, ADC, and GPIO pins are left unconnected."
- moved on the sheet: C3, C5, U2, U4
